Commit message: Add complex indoor capture workflow

File: src/my_robot_description/urdf/robot.urdf.xacro (robot description, xacro)
@@ -269,4 +269,28 @@
     <child link="laser_link"/>
     <origin xyz="0.13 0 0.27" rpy="0 0 0"/>
+  </joint>
+  <link name="imu_link">
+    <visual>
+      <origin xyz="0 0 0" rpy="0 0 0"/>
+      <geometry>
+        <box size="0.035 0.025 0.015"/>
+      </geometry>
+      <material name="gray"/>
+    </visual>
+    <collision>
+      <origin xyz="0 0 0" rpy="0 0 0"/>
+      <geometry>
+        <box size="0.035 0.025 0.015"/>
+      </geometry>
+    </collision>
+    <inertial>
+      <mass value="0.05"/>
+      <inertia ixx="0.00001" ixy="0.0" ixz="0.0" iyy="0.00001" iyz="0.0" izz="0.00001"/>
+    </inertial>
+  </link>
+  <joint name="imu_joint" type="fixed">
+    <parent link="base_link"/>
+    <child link="imu_link"/>
+    <origin xyz="0.0 0.0 0.22" rpy="0 0 0"/>
   </joint>
   <ros2_control name="GazeboSystem" type="system">
@@ -290,11 +314,4 @@
     </plugin>
   </gazebo>
-  <gazebo>
-    <plugin name="front_wheel_joint_state_publisher" filename="libgazebo_ros_joint_state_publisher.so">
-      <update_rate>50</update_rate>
-      <joint_name>front_left_wheel_joint</joint_name>
-      <joint_name>front_right_wheel_joint</joint_name>
-    </plugin>
-  </gazebo>
   <gazebo reference="base_link">
     <material>Gazebo/DarkGrey</material>
@@ -329,16 +346,21 @@
   </gazebo>
   <gazebo>
-    <plugin name="rear_diff_drive_controller" filename="libgazebo_ros_diff_drive.so">
+    <plugin name="skid_steer_drive_controller" filename="libgazebo_ros_diff_drive.so">
       <ros>
         <namespace>/</namespace>
       </ros>
       <update_rate>50</update_rate>
+      <num_wheel_pairs>2</num_wheel_pairs>
+      <left_joint>front_left_wheel_joint</left_joint>
+      <right_joint>front_right_wheel_joint</right_joint>
       <left_joint>rear_left_wheel_joint</left_joint>
       <right_joint>rear_right_wheel_joint</right_joint>
       <wheel_separation>0.36</wheel_separation>
+      <wheel_separation>0.36</wheel_separation>
+      <wheel_diameter>0.16</wheel_diameter>
       <wheel_diameter>0.16</wheel_diameter>
       <max_wheel_torque>10.0</max_wheel_torque>
       <publish_odom>true</publish_odom>
-      <publish_odom_tf>true</publish_odom_tf>
+      <publish_odom_tf>false</publish_odom_tf>
       <publish_wheel_tf>true</publish_wheel_tf>
       <publish_wheel_joint_state>true</publish_wheel_joint_state>
@@ -378,4 +400,53 @@
       </plugin>
     </sensor>
+    <sensor name="lidar3d_sensor" type="ray">
+      <always_on>true</always_on>
+      <visualize>false</visualize>
+      <update_rate>10.0</update_rate>
+      <pose>0 0 0 0 0 0</pose>
+      <ray>
+        <scan>
+          <horizontal>
+            <samples>360</samples>
+            <resolution>1</resolution>
+            <min_angle>-3.14159</min_angle>
+            <max_angle>3.14159</max_angle>
+          </horizontal>
+          <vertical>
+            <samples>16</samples>
+            <resolution>1</resolution>
+            <min_angle>-0.35</min_angle>
+            <max_angle>0.35</max_angle>
+          </vertical>
+        </scan>
+        <range>
+          <min>0.12</min>
+          <max>12.0</max>
+          <resolution>0.02</resolution>
+        </range>
+      </ray>
+      <plugin name="gazebo_ros_lidar3d" filename="libgazebo_ros_ray_sensor.so">
+        <ros>
+          <remapping>~/out:=points_raw</remapping>
+        </ros>
+        <output_type>sensor_msgs/PointCloud2</output_type>
+        <frame_name>laser_link</frame_name>
+      </plugin>
+    </sensor>
+  </gazebo>
+  <gazebo reference="imu_link">
+    <sensor name="imu_sensor" type="imu">
+      <always_on>true</always_on>
+      <visualize>false</visualize>
+      <update_rate>100.0</update_rate>
+      <pose>0 0 0 0 0 0</pose>
+      <plugin name="gazebo_ros_imu" filename="libgazebo_ros_imu_sensor.so">
+        <ros>
+          <remapping>~/out:=imu/data</remapping>
+        </ros>
+        <frame_name>imu_link</frame_name>
+        <initial_orientation_as_reference>false</initial_orientation_as_reference>
+      </plugin>
+    </sensor>
   </gazebo>
   <gazebo reference="camera_link">
